Commit message: fixed the sim and rviz movement

File: src/car_robot_description/urdf/car_robot_gazebo_ros2_control.xacro (robot description, xacro)
@@ -10,4 +10,17 @@
         <origin xyz="${base_length / 4.0} 0 ${base_height}" rpy="0 0 0" />
     </joint> -->
+    <xacro:macro name="wheel_gazebo" params="prefix">
+        <gazebo reference="${prefix}_wheel_link">
+            <mu1>1.0</mu1>
+            <mu2>0.2</mu2>  <!-- Lower lateral friction allows skid-steering turns -->
+            <kp>1000000.0</kp>
+            <kd>10.0</kd>
+            <minDepth>0.001</minDepth>
+        </gazebo>
+    </xacro:macro>
+    <xacro:wheel_gazebo prefix="fl" />
+    <xacro:wheel_gazebo prefix="fr" />
+    <xacro:wheel_gazebo prefix="rl" />
+    <xacro:wheel_gazebo prefix="rr" />
     <joint name="base_lidar_joint" type="fixed">
         <parent link="base_link"/>

Commit message: .

File: src/car_robot_description/urdf/car_robot_gazebo_ros2_control.xacro (robot description, xacro)
@@ -10,17 +10,17 @@
         <origin xyz="${base_length / 4.0} 0 ${base_height}" rpy="0 0 0" />
     </joint> -->
-    <xacro:macro name="wheel_gazebo" params="prefix">
-        <gazebo reference="${prefix}_wheel_link">
-            <mu1>1.0</mu1>
-            <mu2>0.2</mu2>  <!-- Lower lateral friction allows skid-steering turns -->
-            <kp>1000000.0</kp>
-            <kd>10.0</kd>
-            <minDepth>0.001</minDepth>
-        </gazebo>
-    </xacro:macro>
-    <xacro:wheel_gazebo prefix="fl" />
-    <xacro:wheel_gazebo prefix="fr" />
-    <xacro:wheel_gazebo prefix="rl" />
-    <xacro:wheel_gazebo prefix="rr" />
+    <!-- <xacro:macro name="wheel_gazebo" params="prefix">  -->
+        <!-- <gazebo reference="${prefix}_wheel_link"> -->
+            <!-- <mu1>1.0</mu1> -->
+            <!-- <mu2>0.2</mu2>  Lower lateral friction allows skid-steering turns -->
+            <!-- <kp>1000000.0</kp> -->
+            <!-- <kd>10.0</kd> -->
+            <!-- <minDepth>0.001</minDepth> -->
+        <!-- </gazebo> -->
+    <!-- </xacro:macro> -->
+    <!-- <xacro:wheel_gazebo prefix="fl" /> -->
+    <!-- <xacro:wheel_gazebo prefix="fr" /> -->
+    <!-- <xacro:wheel_gazebo prefix="rl" /> -->
+    <!-- <xacro:wheel_gazebo prefix="rr" /> -->
     <joint name="base_lidar_joint" type="fixed">
         <parent link="base_link"/>
