Commit message: new updates

File: src/car_robot_description/urdf/car_base.ros2_control.xacro (robot description, xacro)
@@ -6,24 +6,18 @@
             <plugin>car_base_hardware/CarBaseHardwareInterface</plugin>
             <param name="serial_port">/dev/ttyUSB0</param>
-            <param name="ticks_per_rev">20.0</param>
-            <param name="max_rpm">200.0</param>
-            <!-- <param name="calculate_dynamics">true</param> -->
+            <param name="baud_rate">115200</param>
+            <param name="timeout_ms">500</param>
+            <param name="startup_delay_ms">2000</param>
+            <!-- Optional: velocity PID gains sent to the ESP32 on activation -->
+            <!-- <param name="kp">1.0</param>
+            <param name="ki">0.0</param>
+            <param name="kd">0.0</param> -->
         </hardware>
-        <joint name="base_fl_wheel_joint">
+        <joint name="base_left_wheel_joint">
             <command_interface name="velocity" />
             <state_interface name="velocity" />
             <state_interface name="position" />
         </joint>
-        <joint name="base_fr_wheel_joint">
-            <command_interface name="velocity" />
-            <state_interface name="velocity" />
-            <state_interface name="position" />
-        </joint>
-        <joint name="base_rl_wheel_joint">
-            <command_interface name="velocity" />
-            <state_interface name="velocity" />
-            <state_interface name="position" />
-        </joint>
-        <joint name="base_rr_wheel_joint">
+        <joint name="base_right_wheel_joint">
             <command_interface name="velocity" />
             <state_interface name="velocity" />

File: src/car_robot_description/urdf/car_base.xacro (robot description, xacro)
@@ -1,10 +1,10 @@
 <?xml version="1.0"?>
 <robot xmlns:xacro="http://ros.org/wiki/xacro">
-    <xacro:property name="base_length" value="0.25" />
+    <xacro:property name="base_length" value="0.26" />
     <xacro:property name="base_width" value="0.15" />
     <xacro:property name="base_height" value="0.07" />
     <xacro:property name="wheel_length" value="0.025" />
-    <xacro:property name="wheel_radius" value="0.035" />
-    <!-- <xacro:property name="caster_wheel_radius" value="${wheel_radius / 2.0}" /> -->
+    <xacro:property name="wheel_radius" value="0.0325" />
+    <xacro:property name="caster_wheel_radius" value="${(wheel_radius * 1.5) / 2}" />
     <link name="base_footprint" />
     <link name="base_link">
@@ -40,65 +40,69 @@
                 <origin xyz="0 0 0" rpy="0 0 0" />
             </collision>
-            <xacro:cylinder_inertia m="0.03" r="${wheel_radius}" l="${wheel_length}" o_xyz="0 0 0" o_rpy="${pi / 2.0} 0 0" />
+            <xacro:cylinder_inertia m="0.055" r="${wheel_radius}" l="${wheel_length}" o_xyz="0 0 0" o_rpy="${pi / 2.0} 0 0" />
         </link>
     </xacro:macro>
-    <xacro:wheel_link prefix="fl" />
-    <xacro:wheel_link prefix="fr" />
-    <xacro:wheel_link prefix="rl" />
-    <xacro:wheel_link prefix="rr" />
-    <!-- <link name="caster_wheel_link">
-        <visual>
-            <geometry>
-                <sphere radius="${caster_wheel_radius}"/>
-            </geometry>
-            <origin xyz="0 0 0" rpy="0 0 0"/>
-            <material name="grey" />
-        </visual>
-        <collision>
-            <geometry>
-                <sphere radius="${caster_wheel_radius}"/>
-            </geometry>
-            <origin xyz="0 0 0" rpy="0 0 0"/>
-        </collision>
-        <xacro:sphere_inertia m="0.5" r="${caster_wheel_radius}" o_xyz="0 0 0" o_rpy="0 0 0" />
-    </link> -->
+    <xacro:wheel_link prefix="left" />
+    <xacro:wheel_link prefix="right" />
+    <xacro:macro name="caster_wheel_link" params="prefix">
+        <link name="${prefix}_caster_wheel_link">
+            <visual>
+                <geometry>
+                    <sphere radius="${caster_wheel_radius}"/>
+                </geometry>
+                <origin xyz="0 0 ${-caster_wheel_radius}" rpy="0 0 0"/>
+                <material name="grey" />
+            </visual>
+            <collision>
+                <geometry>
+                    <sphere radius="${caster_wheel_radius}"/>
+                </geometry>
+                <origin xyz="0 0 ${-caster_wheel_radius}" rpy="0 0 0"/>
+            </collision>
+            <xacro:sphere_inertia m="0.037" r="${caster_wheel_radius}" o_xyz="0 0 ${-caster_wheel_radius}" o_rpy="0 0 0" />
+        </link>
+    </xacro:macro>
+    <xacro:caster_wheel_link prefix="fl" />
+    <xacro:caster_wheel_link prefix="fr" />
+    <xacro:caster_wheel_link prefix="rl" />
+    <xacro:caster_wheel_link prefix="rr" />
     <joint name="base_joint" type="fixed">
         <parent link="base_footprint"/>
         <child link="base_link"/>
-        <origin xyz="0 0 ${wheel_radius - (base_height / 3.0)}" rpy="0 0 0"/>
+        <origin xyz="0 0 ${wheel_radius * 1.5}" rpy="0 0 0"/>
     </joint>
-    <joint name="base_fl_wheel_joint" type="continuous">
+    <joint name="base_left_wheel_joint" type="continuous">
         <parent link="base_link" />
-        <child link="fl_wheel_link" />
-        <origin xyz="${base_length / 4.0} ${(base_width + wheel_length) / 2.0} ${base_height / 3.0}" rpy="0 0 0" />
+        <child link="left_wheel_link" />
+        <origin xyz="0 ${((base_width + wheel_length) / 2.0 ) + 0.0075 } ${-(wheel_radius / 2)}" rpy="0 0 0" />
         <axis xyz="0 1 0" />
         <limit effort="100" velocity="100" />
     </joint>
-    <joint name="base_fr_wheel_joint" type="continuous">
+    <joint name="base_right_wheel_joint" type="continuous">
         <parent link="base_link" />
-        <child link="fr_wheel_link" />
-        <origin xyz="${base_length / 4.0} ${-(base_width + wheel_length) / 2.0} ${base_height / 3.0}" rpy="0 0 0" />
+        <child link="right_wheel_link" />
+        <origin xyz="0 ${-(((base_width + wheel_length) / 2.0 ) + 0.0075 )} ${-(wheel_radius / 2)}" rpy="0 0 0" />
         <axis xyz="0 1 0" />
         <limit effort="100" velocity="100" />
     </joint>
-    <joint name="base_rl_wheel_joint" type="continuous">
-        <parent link="base_link" />
-        <child link="rl_wheel_link" />
-        <origin xyz="${-base_length / 4.0} ${(base_width + wheel_length) / 2.0} ${base_height / 3.0}" rpy="0 0 0" />
-        <axis xyz="0 1 0" />
-        <limit effort="100" velocity="100" />
+    <joint name="base_fl_caster_wheel_joint" type="fixed">
+        <parent link="base_link"/>
+        <child link="fl_caster_wheel_link"/>
+        <origin xyz="${(base_length / 2.0) * 0.9} ${base_width / 4} 0" rpy="0 0 0"/>
     </joint>
-    <joint name="base_rr_wheel_joint" type="continuous">
-        <parent link="base_link" />
-        <child link="rr_wheel_link" />
-        <origin xyz="${-base_length / 4.0} ${-(base_width + wheel_length) / 2.0} ${base_height / 3.0}" rpy="0 0 0" />
-        <axis xyz="0 1 0" />
-        <limit effort="100" velocity="100" />
+    <joint name="base_fr_caster_wheel_joint" type="fixed">
+        <parent link="base_link"/>
+        <child link="fr_caster_wheel_link"/>
+        <origin xyz="${(base_length / 2.0) * 0.9} ${-base_width / 4} 0" rpy="0 0 0"/>
     </joint>
-<!--
-    <joint name="base_caster_wheel_joint" type="fixed">
+    <joint name="base_rl_caster_wheel_joint" type="fixed">
         <parent link="base_link"/>
-        <child link="caster_wheel_link"/>
-        <origin xyz="${(base_length / 4.0) * 1.2} 0 ${-caster_wheel_radius}" rpy="0 0 0"/>
-    </joint> -->
+        <child link="rl_caster_wheel_link"/>
+        <origin xyz="${-(base_length / 2.0) * 0.9} ${base_width / 4} 0" rpy="0 0 0"/>
+    </joint>
+    <joint name="base_rr_caster_wheel_joint" type="fixed">
+        <parent link="base_link"/>
+        <child link="rr_caster_wheel_link"/>
+        <origin xyz="${-(base_length / 2.0) * 0.9} ${-base_width / 4} 0" rpy="0 0 0"/>
+    </joint>
 </robot>

File: src/car_robot_description/urdf/car_robot_gazebo_ros2_control.xacro (robot description, xacro)
@@ -10,17 +10,36 @@
         <origin xyz="${base_length / 4.0} 0 ${base_height}" rpy="0 0 0" />
     </joint> -->
-    <!-- <xacro:macro name="wheel_gazebo" params="prefix">  -->
-        <!-- <gazebo reference="${prefix}_wheel_link"> -->
-            <!-- <mu1>1.0</mu1> -->
-            <!-- <mu2>0.2</mu2>  Lower lateral friction allows skid-steering turns -->
-            <!-- <kp>1000000.0</kp> -->
-            <!-- <kd>10.0</kd> -->
-            <!-- <minDepth>0.001</minDepth> -->
-        <!-- </gazebo> -->
-    <!-- </xacro:macro> -->
-    <!-- <xacro:wheel_gazebo prefix="fl" /> -->
-    <!-- <xacro:wheel_gazebo prefix="fr" /> -->
-    <!-- <xacro:wheel_gazebo prefix="rl" /> -->
-    <!-- <xacro:wheel_gazebo prefix="rr" /> -->
+    <!-- Base link -->
+    <gazebo reference="base_link">
+        <material>Gazebo/Blue</material>
+    </gazebo>
+    <!-- Drive wheels: high friction for traction -->
+    <xacro:macro name="wheel_gazebo" params="prefix">
+        <gazebo reference="${prefix}_wheel_link">
+            <mu1>1.0</mu1>
+            <mu2>1.0</mu2>
+            <kp>1000000.0</kp>
+            <kd>100.0</kd>
+            <minDepth>0.001</minDepth>
+            <material>Gazebo/Grey</material>
+        </gazebo>
+    </xacro:macro>
+    <xacro:wheel_gazebo prefix="left" />
+    <xacro:wheel_gazebo prefix="right" />
+    <!-- Caster wheels: near-zero friction so they slide freely -->
+    <xacro:macro name="caster_wheel_gazebo" params="prefix">
+        <gazebo reference="${prefix}_caster_wheel_link">
+            <mu1>0.001</mu1>
+            <mu2>0.001</mu2>
+            <kp>1000000.0</kp>
+            <kd>100.0</kd>
+            <minDepth>0.001</minDepth>
+            <material>Gazebo/Grey</material>
+        </gazebo>
+    </xacro:macro>
+    <xacro:caster_wheel_gazebo prefix="fl" />
+    <xacro:caster_wheel_gazebo prefix="fr" />
+    <xacro:caster_wheel_gazebo prefix="rl" />
+    <xacro:caster_wheel_gazebo prefix="rr" />
     <joint name="base_lidar_joint" type="fixed">
         <parent link="base_link"/>
@@ -32,20 +51,10 @@
             <plugin>gz_ros2_control/GazeboSimSystem</plugin>
         </hardware>
-        <joint name="base_fl_wheel_joint">
+        <joint name="base_left_wheel_joint">
             <command_interface name="velocity" />
             <state_interface name="velocity" />
             <state_interface name="position" />
         </joint>
-        <joint name="base_fr_wheel_joint">
-            <command_interface name="velocity" />
-            <state_interface name="velocity" />
-            <state_interface name="position" />
-        </joint>
-        <joint name="base_rl_wheel_joint">
-            <command_interface name="velocity" />
-            <state_interface name="velocity" />
-            <state_interface name="position" />
-        </joint>
-        <joint name="base_rr_wheel_joint">
+        <joint name="base_right_wheel_joint">
             <command_interface name="velocity" />
             <state_interface name="velocity" />
