Commit message: urdf and slam updates

File: src/car_robot_description/urdf/car_base.xacro (robot description, xacro)
@@ -3,5 +3,5 @@
     <xacro:property name="base_length" value="0.26" />
     <xacro:property name="base_width" value="0.15" />
-    <xacro:property name="base_height" value="0.07" />
+    <xacro:property name="base_height" value="0.08" />
     <xacro:property name="wheel_length" value="0.025" />
     <xacro:property name="wheel_radius" value="0.0325" />
@@ -63,8 +63,6 @@
         </link>
     </xacro:macro>
-    <xacro:caster_wheel_link prefix="fl" />
-    <xacro:caster_wheel_link prefix="fr" />
-    <xacro:caster_wheel_link prefix="rl" />
-    <xacro:caster_wheel_link prefix="rr" />
+    <xacro:caster_wheel_link prefix="front" />
+    <xacro:caster_wheel_link prefix="back" />
     <joint name="base_joint" type="fixed">
         <parent link="base_footprint"/>
@@ -86,23 +84,13 @@
         <limit effort="100" velocity="100" />
     </joint>
-    <joint name="base_fl_caster_wheel_joint" type="fixed">
+    <joint name="base_front_caster_wheel_joint" type="fixed">
         <parent link="base_link"/>
-        <child link="fl_caster_wheel_link"/>
-        <origin xyz="${(base_length / 2.0) * 0.9} ${base_width / 4} 0" rpy="0 0 0"/>
+        <child link="front_caster_wheel_link"/>
+        <origin xyz="${(base_length / 2.0) * 0.7} 0 0" rpy="0 0 0"/>
     </joint>
-    <joint name="base_fr_caster_wheel_joint" type="fixed">
+    <joint name="base_back_caster_wheel_joint" type="fixed">
         <parent link="base_link"/>
-        <child link="fr_caster_wheel_link"/>
-        <origin xyz="${(base_length / 2.0) * 0.9} ${-base_width / 4} 0" rpy="0 0 0"/>
-    </joint>
-    <joint name="base_rl_caster_wheel_joint" type="fixed">
-        <parent link="base_link"/>
-        <child link="rl_caster_wheel_link"/>
-        <origin xyz="${-(base_length / 2.0) * 0.9} ${base_width / 4} 0" rpy="0 0 0"/>
-    </joint>
-    <joint name="base_rr_caster_wheel_joint" type="fixed">
-        <parent link="base_link"/>
-        <child link="rr_caster_wheel_link"/>
-        <origin xyz="${-(base_length / 2.0) * 0.9} ${-base_width / 4} 0" rpy="0 0 0"/>
+        <child link="back_caster_wheel_link"/>
+        <origin xyz="${-(base_length / 2.0)} 0 0" rpy="0 0 0"/>
     </joint>
 </robot>

File: src/car_robot_description/urdf/lidar.xacro (robot description, xacro)
@@ -3,5 +3,5 @@
     <xacro:property name="lidar_length" value="0.1" />
     <xacro:property name="lidar_width" value="0.06" />
-    <xacro:property name="lidar_height" value="0.05" />
+    <xacro:property name="lidar_height" value="0.045" />
     <link name="lidar_link">
         <visual>

Commit message: updated urdf

File: src/car_robot_description/urdf/car_base.xacro (robot description, xacro)
@@ -87,10 +87,10 @@
         <parent link="base_link"/>
         <child link="front_caster_wheel_link"/>
-        <origin xyz="${(base_length / 2.0) * 0.7} 0 0" rpy="0 0 0"/>
+        <origin xyz="${(base_length / 2.0) * 0.8} 0 0" rpy="0 0 0"/>
     </joint>
     <joint name="base_back_caster_wheel_joint" type="fixed">
         <parent link="base_link"/>
         <child link="back_caster_wheel_link"/>
-        <origin xyz="${-(base_length / 2.0)} 0 0" rpy="0 0 0"/>
+        <origin xyz="${-(base_length / 2.0) * 0.6} 0 0" rpy="0 0 0"/>
     </joint>
 </robot>

File: src/car_robot_description/urdf/car_robot.urdf.xacro (robot description, xacro)
@@ -10,5 +10,5 @@
         <parent link="base_link"/>
         <child link="lidar_link"/>
-        <origin xyz="0 0 ${base_height}" rpy="0 0 0"/>
+        <origin xyz="0 0 ${base_height + (lidar_height / 1.5)}" rpy="0 0 0"/>
     </joint>
     <!-- <joint name="mobile_base_arm_joint" type="fixed">

File: src/car_robot_description/urdf/lidar.xacro (robot description, xacro)
@@ -9,5 +9,5 @@
                 <mesh filename="package://car_robot_description/meshes/lds.stl" scale="0.001 0.001 0.001"/>
             </geometry>
-            <origin xyz="0 0 ${lidar_height/1.7}" rpy="0 0 0" />
+            <origin xyz="0 0 ${lidar_height / 16}" rpy="0 0 0" />
             <material name="grey" />
         </visual>
