Commit message: update lidar orientation

File: src/car_robot_description/urdf/car_robot.urdf.xacro (robot description, xacro)
@@ -10,5 +10,5 @@
         <parent link="base_link"/>
         <child link="lidar_link"/>
-        <origin xyz="0 0 ${base_height + (lidar_height / 1.5)}" rpy="0 0 0"/>
+        <origin xyz="0 0 ${base_height + (lidar_height / 1.5)}" rpy="0 0 3.14"/>
     </joint>
     <!-- <joint name="mobile_base_arm_joint" type="fixed">

Commit message: fixed liadar orientation

File: src/car_robot_description/urdf/car_robot.urdf.xacro (robot description, xacro)
@@ -10,5 +10,5 @@
         <parent link="base_link"/>
         <child link="lidar_link"/>
-        <origin xyz="0 0 ${base_height + (lidar_height / 1.5)}" rpy="0 0 0"/>
+        <origin xyz="0 0 ${base_height + (lidar_height / 1.5)}" rpy="0 0 ${pi}"/>
     </joint>
     <!-- <joint name="mobile_base_arm_joint" type="fixed">

Commit message: fixed the inversion in the lidar

File: src/car_robot_description/urdf/car_robot.urdf.xacro (robot description, xacro)
@@ -10,5 +10,5 @@
         <parent link="base_link"/>
         <child link="lidar_link"/>
-        <origin xyz="0 0 ${base_height + (lidar_height / 1.5)}" rpy="0 0 ${pi}"/>
+        <origin xyz="0 0 ${base_height + (lidar_height / 1.5)}" rpy="0 0 0"/>
     </joint>
     <!-- <joint name="mobile_base_arm_joint" type="fixed">
