Commit message: arm in prgress and return lidar position

File: src/car_robot_description/urdf/arm.xacro (robot description, xacro)
@@ -3,9 +3,19 @@
     <xacro:property name="arm_base_length" value="0.1" />
     <xacro:property name="arm_base_width" value="0.1" />
-    <xacro:property name="arm_base_height" value="0.02" />
-    <xacro:property name="forearm_radius" value="0.02" />
-    <xacro:property name="forearm_length" value="0.3" />
-    <xacro:property name="hand_radius" value="0.02" />
-    <xacro:property name="hand_length" value="0.3" />
+    <xacro:property name="arm_base_height" value="0.025" />
+    <xacro:property name="arm_shoulder_radius" value="0.0125" />
+    <xacro:property name="arm_shoulder_length" value="0.025" />
+    <xacro:property name="arm_upper_arm_radius" value="0.15" />
+    <xacro:property name="arm_upper_arm_length" value="0.0125" />
+    <xacro:property name="arm_elbow_radius" value="0.025" />
+    <xacro:property name="arm_elbow_length" value="0.0125" />
+    <xacro:property name="arm_forearm_radius" value="0.125" />
+    <xacro:property name="arm_forearm_length" value="0.0125" />
+    <xacro:property name="arm_wrist_length" value="0.025" />
+    <xacro:property name="arm_wrist_width" value="0.025" />
+    <xacro:property name="arm_wrist_height" value="0.0125" />
+    <xacro:property name="arm_hand_length" value="0.025" />
+    <xacro:property name="arm_hand_width" value="0.025" />
+    <xacro:property name="arm_hand_height" value="0.005" />
     <link name="arm_base_link">
         <visual>
@@ -17,37 +27,110 @@
         </visual>
     </link>
-    <link name="forearm_link">
+    <link name="arm_shoulder_link">
         <visual>
             <geometry>
-                <cylinder radius="${forearm_radius}" length="${forearm_length}" />
+                <cylinder radius="${arm_shoulder_radius}" length="${arm_shoulder_length}" />
             </geometry>
-            <origin xyz="0 0 ${forearm_length / 2.0}" rpy="0 0 0" />
+            <origin xyz="0 0 ${arm_shoulder_length / 2.0}" rpy="0 0 0" />
             <material name="yellow" />
         </visual>
     </link>
-    <link name="hand_link">
+    <link name="arm_upper_arm_link">
         <visual>
             <geometry>
-                <cylinder radius="${hand_radius}" length="${hand_length}" />
+                <cylinder radius="${arm_upper_arm_radius}" length="${arm_upper_arm_length}" />
             </geometry>
-            <origin xyz="0 0 ${hand_length / 2.0}" rpy="0 0 0" />
+            <origin xyz="0 0 ${arm_upper_arm_length / 2.0}" rpy="0 0 0" />
             <material name="orange" />
         </visual>
     </link>
+    <link name="arm_elbow_link">
+        <visual>
+            <geometry>
+                <cylinder radius="${arm_elbow_radius}" length="${arm_elbow_length}" />
+            </geometry>
+            <origin xyz="0 0 ${arm_elbow_length / 2.0}" rpy="0 0 0" />
+            <material name="orange" />
+        </visual>
+    </link>
+    <link name="arm_forearm_link">
+        <visual>
+            <geometry>
+                <cylinder radius="${arm_forearm_radius}" length="${arm_forearm_length}" />
+            </geometry>
+            <origin xyz="0 0 ${arm_forearm_length / 2.0}" rpy="0 0 0" />
+            <material name="orange" />
+        </visual>
+    </link>
+    <link name="arm_wrist_link">
+        <visual>
+            <geometry>
+                <box size="${arm_wrist_length} ${arm_wrist_width} ${arm_wrist_height}"/>
+            </geometry>
+            <origin xyz="0 0 ${arm_wrist_height / 2.0}" rpy="0 0 0" />
+            <material name="orange" />
+        </visual>
+    </link>
+    <link name="arm_hand_link">
+        <visual>
+            <geometry>
+                <box size="${arm_hand_length} ${arm_hand_width} ${arm_hand_height}"/>
+            </geometry>
+            <origin xyz="0 0 ${arm_hand_height / 2.0}" rpy="0 0 0" />
+            <material name="orange" />
+        </visual>
+    </link>
+    <link name="arm_tool_link" />
     <joint name="arm_joint1" type="revolute">
         <parent link="arm_base_link" />
-        <child link="forearm_link" />
+        <child link="arm_shoulder_link" />
         <origin xyz="0 0 ${arm_base_height}" rpy="0 0 0" />
-        <axis xyz="0 1 0" />
-        <limit lower="0" upper="${pi/2}" effort="100" velocity="100" />
+        <axis xyz="0 0 1" />
+        <limit lower="${-pi}" upper="${pi}" effort="100" velocity="100" />
         <dynamics friction="0.05" damping="0.1" />
     </joint>
     <joint name="arm_joint2" type="revolute">
-        <parent link="forearm_link" />
-        <child link="hand_link" />
-        <origin xyz="0 0 ${forearm_length}" rpy="0 0 0" />
+        <parent link="arm_shoulder_link" />
+        <child link="arm_upper_arm_link" />
+        <origin xyz="0 0 ${arm_shoulder_length}" rpy="0 0 0" />
         <axis xyz="0 1 0" />
-        <limit lower="0" upper="${pi/2}" effort="100" velocity="100" />
+        <limit lower="0" upper="2.5" effort="100" velocity="100" />
         <dynamics friction="0.05" damping="0.1" />
     </joint>
+    <joint name="arm_joint3" type="revolute">
+        <parent link="arm_upper_arm_link" />
+        <child link="arm_elbow_link" />
+        <origin xyz="0 0 ${arm_upper_arm_length}" rpy="0 0 0" />
+        <axis xyz="0 1 0" />
+        <limit lower="0" upper="2.5" effort="100" velocity="100" />
+        <dynamics friction="0.05" damping="0.1" />
+    </joint>
+    <joint name="arm_joint4" type="revolute">
+        <parent link="arm_elbow_link" />
+        <child link="arm_forearm_link" />
+        <origin xyz="0 0 ${arm_elbow_length}" rpy="0 0 0" />
+        <axis xyz="0 0 1" />
+        <limit lower="${-pi}" upper="${pi}" effort="100" velocity="100" />
+        <dynamics friction="0.05" damping="0.1" />
+    </joint>
+    <joint name="arm_joint5" type="revolute">
+        <parent link="arm_forearm_link" />
+        <child link="arm_wrist_link" />
+        <origin xyz="0 0 ${arm_forearm_length}" rpy="0 0 0" />
+        <axis xyz="0 1 0" />
+        <limit lower="${-pi/2}" upper="${pi/2}" effort="100" velocity="100" />
+        <dynamics friction="0.05" damping="0.1" />
+    </joint>
+    <joint name="arm_joint6" type="continuous">
+        <parent link="arm_wrist_link" />
+        <child link="arm_hand_link" />
+        <origin xyz="0 0 ${arm_wrist_height}" rpy="0 0 0" />
+        <axis xyz="0 0 1" />
+        <dynamics friction="0.05" damping="0.1" />
+    </joint>
+    <joint name="arm_joint7" type="fixed">
+        <parent link="arm_hand_link" />
+        <child link="arm_tool_link" />
+        <origin xyz="0 0 ${arm_hand_height}" rpy="0 0 0" />
+    </joint>
 </robot>

File: src/car_robot_description/urdf/car_robot.urdf.xacro (robot description, xacro)
@@ -10,5 +10,5 @@
         <parent link="base_link"/>
         <child link="lidar_link"/>
-        <origin xyz="0 0 ${base_height + (lidar_height / 1.5)}" rpy="0 0 3.14"/>
+        <origin xyz="0 0 ${base_height + (lidar_height / 1.5)}" rpy="0 0 0"/>
     </joint>
     <!-- <joint name="mobile_base_arm_joint" type="fixed">

Commit message: added robotics arm in urdf and created the moveit config

File: src/car_robot_description/urdf/arm.xacro (robot description, xacro)
@@ -1,15 +1,15 @@
 <?xml version="1.0"?>
-<robot xmlns:xacro="http://www.ros.org/wiki/xacro">
+<robot xmlns:xacro="http://www.ros.org/wiki/xacro"> # name="arm"
     <xacro:property name="arm_base_length" value="0.1" />
     <xacro:property name="arm_base_width" value="0.1" />
     <xacro:property name="arm_base_height" value="0.025" />
-    <xacro:property name="arm_shoulder_radius" value="0.0125" />
-    <xacro:property name="arm_shoulder_length" value="0.025" />
-    <xacro:property name="arm_upper_arm_radius" value="0.15" />
-    <xacro:property name="arm_upper_arm_length" value="0.0125" />
-    <xacro:property name="arm_elbow_radius" value="0.025" />
-    <xacro:property name="arm_elbow_length" value="0.0125" />
-    <xacro:property name="arm_forearm_radius" value="0.125" />
-    <xacro:property name="arm_forearm_length" value="0.0125" />
+    <xacro:property name="arm_shoulder_radius" value="0.0250" />
+    <xacro:property name="arm_shoulder_length" value="0.125" />
+    <xacro:property name="arm_upper_arm_radius" value="0.0125" />
+    <xacro:property name="arm_upper_arm_length" value="0.15" />
+    <xacro:property name="arm_elbow_radius" value="0.0125" />
+    <xacro:property name="arm_elbow_length" value="0.025" />
+    <xacro:property name="arm_forearm_radius" value="0.0125" />
+    <xacro:property name="arm_forearm_length" value="0.125" />
     <xacro:property name="arm_wrist_length" value="0.025" />
     <xacro:property name="arm_wrist_width" value="0.025" />
@@ -24,6 +24,12 @@
             </geometry>
             <origin xyz="0 0 ${arm_base_height / 2.0}" rpy="0 0 0" />
-            <material name="orange" />
+            <material name="grey" />
         </visual>
+        <collision>
+            <geometry>
+                <box size="${arm_base_length} ${arm_base_width} ${arm_base_height}" />
+            </geometry>
+            <origin xyz="0 0 ${arm_base_height / 2.0}" rpy="0 0 0" />
+        </collision>
     </link>
     <link name="arm_shoulder_link">
@@ -33,6 +39,12 @@
             </geometry>
             <origin xyz="0 0 ${arm_shoulder_length / 2.0}" rpy="0 0 0" />
-            <material name="yellow" />
+            <material name="blue" />
         </visual>
+        <collision>
+            <geometry>
+                <cylinder radius="${arm_shoulder_radius}" length="${arm_shoulder_length}" />
+            </geometry>
+            <origin xyz="0 0 ${arm_shoulder_length / 2.0}" rpy="0 0 0" />
+        </collision>
     </link>
     <link name="arm_upper_arm_link">
@@ -42,6 +54,12 @@
             </geometry>
             <origin xyz="0 0 ${arm_upper_arm_length / 2.0}" rpy="0 0 0" />
-            <material name="orange" />
+            <material name="grey" />
         </visual>
+        <collision>
+            <geometry>
+                <cylinder radius="${arm_upper_arm_radius}" length="${arm_upper_arm_length}" />
+            </geometry>
+            <origin xyz="0 0 ${arm_upper_arm_length / 2.0}" rpy="0 0 0" />
+        </collision>
     </link>
     <link name="arm_elbow_link">
@@ -51,6 +69,12 @@
             </geometry>
             <origin xyz="0 0 ${arm_elbow_length / 2.0}" rpy="0 0 0" />
-            <material name="orange" />
+            <material name="blue" />
         </visual>
+        <collision>
+            <geometry>
+                <cylinder radius="${arm_elbow_radius}" length="${arm_elbow_length}" />
+            </geometry>
+            <origin xyz="0 0 ${arm_elbow_length / 2.0}" rpy="0 0 0" />
+        </collision>
     </link>
     <link name="arm_forearm_link">
@@ -60,6 +84,12 @@
             </geometry>
             <origin xyz="0 0 ${arm_forearm_length / 2.0}" rpy="0 0 0" />
-            <material name="orange" />
+            <material name="grey" />
         </visual>
+        <collision>
+            <geometry>
+                <cylinder radius="${arm_forearm_radius}" length="${arm_forearm_length}" />
+            </geometry>
+            <origin xyz="0 0 ${arm_forearm_length / 2.0}" rpy="0 0 0" />
+        </collision>
     </link>
     <link name="arm_wrist_link">
@@ -69,6 +99,12 @@
             </geometry>
             <origin xyz="0 0 ${arm_wrist_height / 2.0}" rpy="0 0 0" />
-            <material name="orange" />
+            <material name="blue" />
         </visual>
+        <collision>
+            <geometry>
+                <box size="${arm_wrist_length} ${arm_wrist_width} ${arm_wrist_height}"/>
+            </geometry>
+            <origin xyz="0 0 ${arm_wrist_height / 2.0}" rpy="0 0 0" />
+        </collision>
     </link>
     <link name="arm_hand_link">
@@ -78,8 +114,14 @@
             </geometry>
             <origin xyz="0 0 ${arm_hand_height / 2.0}" rpy="0 0 0" />
-            <material name="orange" />
+            <material name="grey" />
         </visual>
+        <collision>
+            <geometry>
+                <box size="${arm_hand_length} ${arm_hand_width} ${arm_hand_height}"/>
+            </geometry>
+            <origin xyz="0 0 ${arm_hand_height / 2.0}" rpy="0 0 0" />
+        </collision>
     </link>
-    <link name="arm_tool_link" />
+    <link name="tool0" />
     <joint name="arm_joint1" type="revolute">
         <parent link="arm_base_link" />
@@ -129,7 +171,7 @@
         <dynamics friction="0.05" damping="0.1" />
     </joint>
-    <joint name="arm_joint7" type="fixed">
+    <joint name="hand_tool_joint" type="fixed">
         <parent link="arm_hand_link" />
-        <child link="arm_tool_link" />
+        <child link="tool0" />
         <origin xyz="0 0 ${arm_hand_height}" rpy="0 0 0" />
     </joint>

File: src/car_robot_description/urdf/car_base.ros2_control.xacro (robot description, xacro)
@@ -3,10 +3,10 @@
     <ros2_control name="CarRobotHardwareInterface" type="system">
         <hardware>
-            <!-- <plugin>mock_components/GenericSystem</plugin> -->
-            <plugin>car_base_hardware/CarBaseHardwareInterface</plugin>
+            <plugin>mock_components/GenericSystem</plugin>
+            <!-- <plugin>car_base_hardware/CarBaseHardwareInterface</plugin>
             <param name="serial_port">/dev/esp32</param>
             <param name="baud_rate">115200</param>
             <param name="timeout_ms">500</param>
-            <param name="startup_delay_ms">2000</param>
+            <param name="startup_delay_ms">2000</param> -->
             <!-- Optional - velocity PID gains sent to the ESP32 on activation -->
             <!-- <param name="kp">1.0</param>

File: src/car_robot_description/urdf/car_robot.urdf.xacro (robot description, xacro)
@@ -5,15 +5,21 @@
     <xacro:include filename="car_base.ros2_control.xacro"/>
     <xacro:include filename="lidar.xacro"/>
-    <!-- <xacro:include filename="arm.xacro"/>
-    <xacro:include filename="arm.ros2_control.xacro"/> -->
+    <xacro:include filename="arm.xacro"/>
+    <xacro:include filename="gripper.xacro"/>
+    <xacro:include filename="car_arm.ros2_control.xacro"/>
     <joint name="base_lidar_joint" type="fixed">
         <parent link="base_link"/>
         <child link="lidar_link"/>
-        <origin xyz="0 0 ${base_height + (lidar_height / 1.5)}" rpy="0 0 0"/>
+        <origin xyz="${base_length / 5.0} 0 ${base_height + (lidar_height / 1.5)}" rpy="0 0 0"/>
     </joint>
-    <!-- <joint name="mobile_base_arm_joint" type="fixed">
+    <joint name="base_arm_joint" type="fixed">
         <parent link="base_link" />
         <child link="arm_base_link" />
-        <origin xyz="${base_length / 4.0} 0 ${base_height}" rpy="0 0 0" />
-    </joint> -->
+        <origin xyz="${-base_length / 4.0} 0 ${base_height}" rpy="0 0 0" />
+    </joint>
+    <joint name="arm_hand_gripper_joint" type="fixed">
+        <parent link="tool0" />
+        <child link="gripper_base_link" />
+        <origin xyz="0 0 0" rpy="0 0 0" />
+    </joint>
 </robot>

File: src/car_robot_description/urdf/car_robot_gazebo_ros2_control.xacro (robot description, xacro)
@@ -65,5 +65,5 @@
         <!-- Actuators & Wheel Control -->
         <plugin filename="gz_ros2_control-system" name="gz_ros2_control::GazeboSimROS2ControlPlugin">
-            <parameters>$(find car_robot_bringup)/config/my_robot_controller.yaml</parameters>
+            <parameters>$(find car_robot_bringup)/config/car_robot_controller.yaml</parameters>
         </plugin>
         <!-- GPU LiDAR & Camera Rendering Engine -->

File: src/car_robot_description/urdf/lidar.xacro (robot description, xacro)
@@ -16,4 +16,5 @@
                 <box size="${lidar_length} ${lidar_width} ${lidar_height}"/>
             </geometry>
+            <origin xyz="0 0 ${lidar_height / 16}" rpy="0 0 0" />
         </collision>
         <xacro:box_inertia m="0.13" x="${lidar_length}" y="${lidar_width}" z="${lidar_height}"
